File: ocxo.kicad_pcb (KiCad board)
At the start: 2 copper layers, 50 x 50 mm, 501 parts, among them J1 Conn_01x02, J2 Conn_01x01, J3 Conn_Coaxial, J4 Conn_01x01, J5 Conn_01x01, J6 Conn_01x01, J7 Conn_Coaxial, Q1 ENE3311 OCXO, U1 KA78M05_TO252, U2 LM4140

Commit message: sma cleaning
Changed lines of the file:
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@@
     (links 526)
     (no_connects 0)
-    (area 79.157143 44.025 131.842858 104.275001)
+    (area 79.924999 44.924999 130.075001 95.075001)
     (thickness 1.6)
     (drawings 9)
@@
     (effects (font (size 1.5 1.5) (thickness 0.3)) (justify right))
   )
-  (gr_text "10 MHz OCXO \nFrequency Reference\n" (at 90 87 90) (layer F.SilkS)
-    (effects (font (size 1.5 1.5) (thickness 0.3) italic) (justify left))
+  (gr_text "10 MHz OCXO \nFrequency Reference\n" (at 90.75 71.5 90) (layer F.SilkS)
+    (effects (font (size 1.5 1.5) (thickness 0.3) italic))
   )
   (gr_text "Vcc In\n++ 7/12V" (at 124.5 66 90) (layer F.SilkS)
