File: ocxo.kicad_pcb (KiCad board)
At the start: 2 copper layers, 50 x 50 mm, 658 parts, among them J1 Conn_01x02, J2 Conn_01x01, J3 Conn_Coaxial, J4 Conn_01x01, J5 Conn_01x01, J6 Conn_01x01, J7 Conn_Coaxial, Q1 ENE3311 OCXO, U1 KA78M05_TO252, U2 LM4140

Commit message: new gerber, minor changes on the output stripline
Parts:
- removed the REF** at (127.0, 85.0)
- removed the REF** at (126.0, 85.0)
- removed the REF** at (125.0, 85.0)
- removed the REF** at (124.0, 85.0)
- removed the REF** at (127.0, 84.0)
- removed the REF** at (126.0, 84.0)
- removed the REF** at (125.0, 84.0)
- removed the REF** at (124.0, 84.0)
- removed the REF** at (127.0, 83.0)
- removed the REF** at (126.0, 83.0)
- removed the REF** at (125.0, 83.0)
- removed the REF** at (124.0, 83.0)
- removed the REF** at (127.0, 82.0)
- removed the REF** at (126.0, 82.0)
- removed the REF** at (125.0, 82.0)
- removed the REF** at (124.0, 82.0)
- removed the REF** at (127.0, 81.0)
- removed the REF** at (126.0, 81.0)
- removed the REF** at (125.0, 81.0)
- removed the REF** at (124.0, 81.0)
- removed the REF** at (127.0, 80.0)
- removed the REF** at (126.0, 80.0)
- removed the REF** at (125.0, 80.0)
- removed the REF** at (124.0, 80.0)
- removed the REF** at (127.0, 79.0)
- removed the REF** at (126.0, 79.0)
- removed the REF** at (125.0, 79.0)
- removed the REF** at (124.0, 79.0)
- removed the REF** at (127.0, 78.0)
- removed the REF** at (126.0, 78.0)
- removed the REF** at (125.0, 78.0)
- removed the REF** at (124.0, 78.0)
- removed the REF** at (127.0, 77.0)
- removed the REF** at (126.0, 77.0)
- removed the REF** at (125.0, 77.0)
- removed the REF** at (124.0, 77.0)
- removed the REF** at (127.0, 76.0)
- removed the REF** at (126.0, 76.0)
- removed the REF** at (125.0, 76.0)
- removed the REF** at (124.0, 76.0)
- removed the REF** at (93.0, 92.0)
- removed the REF** at (92.0, 92.0)
- removed the REF** at (91.0, 92.0)
- removed the REF** at (90.0, 92.0)
- removed the REF** at (93.0, 91.0)
- removed the REF** at (92.0, 91.0)
- removed the REF** at (91.0, 91.0)
- removed the REF** at (90.0, 91.0)
- removed the REF** at (93.0, 90.0)
- removed the REF** at (92.0, 90.0)
- removed the REF** at (91.0, 90.0)
- removed the REF** at (90.0, 90.0)
- removed the REF** at (109.0, 92.0)
- removed the REF** at (108.0, 92.0)
- removed the REF** at (107.0, 92.0)
- removed the REF** at (109.0, 91.0)
- removed the REF** at (108.0, 91.0)
- removed the REF** at (107.0, 91.0)
- removed the REF** at (109.0, 90.0)
- removed the REF** at (108.0, 90.0)
- removed the REF** at (107.0, 90.0)
- removed the REF** at (109.0, 89.0)
- removed the REF** at (108.0, 89.0)
- removed the REF** at (107.0, 89.0)
- removed the REF** at (109.0, 88.0)
- removed the REF** at (108.0, 88.0)
- removed the REF** at (107.0, 88.0)
- removed the REF** at (85.0, 84.0)
- removed the REF** at (84.0, 84.0)
- removed the REF** at (83.0, 84.0)
- removed the REF** at (85.0, 83.0)
- removed the REF** at (84.0, 83.0)
- removed the REF** at (83.0, 83.0)
- removed the REF** at (85.0, 82.0)
- removed the REF** at (84.0, 82.0)
- removed the REF** at (83.0, 82.0)
- removed the REF** at (85.0, 81.0)
- removed the REF** at (84.0, 81.0)
- removed the REF** at (83.0, 81.0)
- removed the REF** at (85.0, 80.0)
- removed the REF** at (84.0, 80.0)
- removed the REF** at (83.0, 80.0)
- removed the REF** at (85.0, 79.0)
- removed the REF** at (84.0, 79.0)
- removed the REF** at (83.0, 79.0)
- removed the REF** at (85.0, 78.0)
- removed the REF** at (84.0, 78.0)
- removed the REF** at (83.0, 78.0)
- removed the REF** at (85.0, 77.0)
- removed the REF** at (84.0, 77.0)
- removed the REF** at (83.0, 77.0)
- removed the REF** at (85.0, 76.0)
- removed the REF** at (84.0, 76.0)
- removed the REF** at (83.0, 76.0)
- removed the REF** at (85.0, 75.0)
- removed the REF** at (84.0, 75.0)
- removed the REF** at (83.0, 75.0)
- removed the REF** at (85.0, 74.0)
- removed the REF** at (84.0, 74.0)
- removed the REF** at (83.0, 74.0)
- removed the REF** at (85.0, 73.0)
- removed the REF** at (84.0, 73.0)
- removed the REF** at (83.0, 73.0)
- removed the REF** at (85.0, 72.0)
- removed the REF** at (84.0, 72.0)
- removed the REF** at (83.0, 72.0)
- removed the REF** at (85.0, 71.0)
- removed the REF** at (84.0, 71.0)
- removed the REF** at (83.0, 71.0)
- removed the REF** at (85.0, 70.0)
- removed the REF** at (84.0, 70.0)
- removed the REF** at (83.0, 70.0)
- removed the REF** at (85.0, 69.0)
- removed the REF** at (84.0, 69.0)
- removed the REF** at (83.0, 69.0)
- removed the REF** at (85.0, 68.0)
- removed the REF** at (84.0, 68.0)
- removed the REF** at (83.0, 68.0)
- removed the REF** at (85.0, 67.0)
- removed the REF** at (84.0, 67.0)
- removed the REF** at (83.0, 67.0)
- removed the REF** at (85.0, 66.0)
- removed the REF** at (84.0, 66.0)
- removed the REF** at (83.0, 66.0)
- removed the REF** at (85.0, 65.0)
- removed the REF** at (84.0, 65.0)
- removed the REF** at (83.0, 65.0)
- removed the REF** at (85.0, 64.0)
- removed the REF** at (84.0, 64.0)
- removed the REF** at (83.0, 64.0)
- removed the REF** at (85.0, 63.0)
- removed the REF** at (84.0, 63.0)
- removed the REF** at (83.0, 63.0)
- removed the REF** at (85.0, 62.0)
- removed the REF** at (84.0, 62.0)
- removed the REF** at (83.0, 62.0)
- removed the REF** at (85.0, 61.0)
- removed the REF** at (84.0, 61.0)
- removed the REF** at (83.0, 61.0)
- removed the REF** at (85.0, 60.0)
- removed the REF** at (84.0, 60.0)
- removed the REF** at (83.0, 60.0)
- removed the REF** at (85.0, 59.0)
- removed the REF** at (84.0, 59.0)
- removed the REF** at (83.0, 59.0)
- removed the REF** at (85.0, 58.0)
- removed the REF** at (84.0, 58.0)
- removed the REF** at (83.0, 58.0)
- removed the REF** at (85.0, 57.0)
- removed the REF** at (84.0, 57.0)
- removed the REF** at (83.0, 57.0)
- removed the REF** at (85.0, 56.0)
- removed the REF** at (84.0, 56.0)
- removed the REF** at (83.0, 56.0)
- removed the REF** at (85.0, 55.0)
- removed the REF** at (84.0, 55.0)
- removed the REF** at (83.0, 55.0)
Routing:
- net GND: vias 55 -> 54

Commit message: minor bug fixed
Routing:
- net GND: track 108.2 -> 106.2 mm
Other:
- board text added: "10 MHz OCXO Frequency Reference (v1)"
- board text removed: "10 MHz OCXO Frequency Reference"
Changed lines of the file:
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@@
     (links 526)
     (no_connects 0)
-    (area 79.924999 44.924999 130.075001 95.075001)
+    (area 79.157143 44.025 131.842858 104.275001)
     (thickness 1.6)
     (drawings 9)
-    (tracks 182)
+    (tracks 181)
     (zones 0)
     (modules 501)
@@
     (mod_text_size 1 1)
     (mod_text_width 0.15)
-    (pad_size 0.6 0.6)
-    (pad_drill 0.3)
+    (pad_size 2.5 2.5)
+    (pad_drill 1)
     (pad_to_mask_clearance 0.2)
     (aux_axis_origin 0 0)
@@
     (fp_arc (start 11.43 11.43) (end 12.7 11.43) (angle 90) (layer F.SilkS) (width 0.4))
     (fp_line (start -12.7 12.7) (end 11.43 12.7) (layer F.SilkS) (width 0.4))
-    (pad 5 thru_hole circle (at -9.525 -9.525) (size 2.5 2.5) (drill 0.8) (layers *.Cu *.Mask)
+    (pad 5 thru_hole circle (at -9.525 -9.525) (size 2.5 2.5) (drill 1) (layers *.Cu *.Mask)
       (net 3 "Net-(C2-Pad1)"))
-    (pad 4 thru_hole circle (at 9.525 -9.525) (size 2.5 2.5) (drill 0.8) (layers *.Cu *.Mask))
-    (pad 3 thru_hole circle (at 9.525 9.525) (size 2.5 2.5) (drill 0.8) (layers *.Cu *.Mask)
+    (pad 4 thru_hole circle (at 9.525 -9.525) (size 2.5 2.5) (drill 1) (layers *.Cu *.Mask))
+    (pad 3 thru_hole circle (at 9.525 9.525) (size 2.5 2.5) (drill 1) (layers *.Cu *.Mask)
       (net 4 "Net-(C4-Pad1)"))
-    (pad 1 thru_hole circle (at -9.525 9.525) (size 2.5 2.5) (drill 0.8) (layers *.Cu *.Mask)
+    (pad 1 thru_hole circle (at -9.525 9.525) (size 2.5 2.5) (drill 1) (layers *.Cu *.Mask)
       (net 6 "Net-(J3-Pad1)"))
-    (pad 2 thru_hole circle (at 0 9.525) (size 2.5 2.5) (drill 0.8) (layers *.Cu *.Mask)
+    (pad 2 thru_hole circle (at 0 9.525) (size 2.5 2.5) (drill 1) (layers *.Cu *.Mask)
       (net 2 GND))
     (model ../../../../../../Users/Marco/Documents/Kicad/modules/ENE3311.pretty/ENE3311.wrl
@@
     (effects (font (size 1.5 1.5) (thickness 0.3)) (justify right))
   )
-  (gr_text "10 MHz OCXO \nFrequency Reference\n" (at 90 87 90) (layer F.SilkS)
+  (gr_text "10 MHz OCXO \nFrequency Reference (v1)\n" (at 90 87 90) (layer F.SilkS)
     (effects (font (size 1.5 1.5) (thickness 0.3) italic) (justify left))
   )
@@
   (segment (start 111.5 55) (end 111.5 57) (width 0.25) (layer B.Cu) (net 2))
   (via (at 111.5 57) (size 0.6) (drill 0.4) (layers F.Cu B.Cu) (net 2))
-  (segment (start 84 91) (end 86 91) (width 0.25) (layer B.Cu) (net 2))
   (segment (start 126 49) (end 124 49) (width 0.25) (layer F.Cu) (net 2))
   (segment (start 126 91) (end 126 89) (width 0.25) (layer B.Cu) (net 2))
@@
   (segment (start 123.3 55.3) (end 120 55.3) (width 1.5) (layer B.Cu) (net 5))
   (segment (start 125.25 57.25) (end 123.3 55.3) (width 1.5) (layer B.Cu) (net 5))
+  (segment (start 100 90) (end 100 93) (width 1.5) (layer F.Cu) (net 6))
   (segment (start 100 90) (end 100 83.4) (width 2) (layer F.Cu) (net 6))
   (segment (start 100 83.4) (end 97.4 80.8) (width 2) (layer F.Cu) (net 6))
   (segment (start 97.4 80.8) (end 97.4 69.6) (width 2) (layer F.Cu) (net 6))
   (segment (start 97.4 69.6) (end 97.475 69.525) (width 2) (layer F.Cu) (net 6))
-  (segment (start 100 93) (end 100 90) (width 1.5) (layer F.Cu) (net 6))
   (segment (start 107.635 82.175) (end 107.635 80.365) (width 0.6) (layer B.Cu) (net 7))
   (segment (start 108.65 79.35) (end 108 80) (width 1) (layer B.Cu) (net 7))

Commit message: small mods on stitching
Parts:
- removed J4: Conn_01x01, MountingHole:MountingHole_3.2mm_M3_ISO14580_Pad
- removed J7: Conn_Coaxial, SMA_PINS:SMA_EDGE_NRW
- removed the REF** at (93.0, 48.0)
- removed the REF** at (92.0, 48.0)
- removed the REF** at (91.0, 48.0)
- removed the REF** at (90.0, 48.0)
- removed the REF** at (89.0, 48.0)
- removed the REF** at (88.0, 48.0)
- removed the REF** at (127.0, 87.0)
- removed the REF** at (126.0, 87.0)
- removed the REF** at (125.0, 87.0)
- removed the REF** at (124.0, 87.0)
- removed the REF** at (123.0, 87.0)
- removed the REF** at (122.0, 87.0)
- removed the REF** at (127.0, 86.0)
- removed the REF** at (126.0, 86.0)
- removed the REF** at (125.0, 86.0)
- removed the REF** at (124.0, 86.0)
- removed the REF** at (123.0, 86.0)
- removed the REF** at (122.0, 86.0)
- removed the REF** at (123.0, 85.0)
- removed the REF** at (122.0, 85.0)
- removed the REF** at (123.0, 84.0)
- removed the REF** at (122.0, 84.0)
- removed the REF** at (123.0, 83.0)
- removed the REF** at (122.0, 83.0)
- removed the REF** at (123.0, 82.0)
- removed the REF** at (122.0, 82.0)
- removed the REF** at (123.0, 81.0)
- removed the REF** at (122.0, 81.0)
- removed the REF** at (123.0, 80.0)
- removed the REF** at (122.0, 80.0)
- removed the REF** at (123.0, 79.0)
- removed the REF** at (122.0, 79.0)
- removed the REF** at (123.0, 78.0)
- removed the REF** at (122.0, 78.0)
- removed the REF** at (123.0, 77.0)
- removed the REF** at (122.0, 77.0)
- removed the REF** at (123.0, 76.0)
- removed the REF** at (122.0, 76.0)
- removed the REF** at (127.0, 75.0)
- removed the REF** at (126.0, 75.0)
- removed the REF** at (125.0, 75.0)
- removed the REF** at (124.0, 75.0)
- removed the REF** at (123.0, 75.0)
- removed the REF** at (122.0, 75.0)
- removed the REF** at (127.0, 74.0)
- removed the REF** at (126.0, 74.0)
- removed the REF** at (125.0, 74.0)
- removed the REF** at (124.0, 74.0)
- removed the REF** at (123.0, 74.0)
- removed the REF** at (95.0, 92.0)
- removed the REF** at (94.0, 92.0)
- removed the REF** at (89.0, 92.0)
- removed the REF** at (88.0, 92.0)
- removed the REF** at (95.0, 91.0)
- removed the REF** at (94.0, 91.0)
- removed the REF** at (89.0, 91.0)
- removed the REF** at (88.0, 91.0)
- removed the REF** at (95.0, 90.0)
- removed the REF** at (94.0, 90.0)
- removed the REF** at (89.0, 90.0)
- removed the REF** at (88.0, 90.0)
- removed the REF** at (95.0, 89.0)
- removed the REF** at (94.0, 89.0)
- removed the REF** at (93.0, 89.0)
- removed the REF** at (92.0, 89.0)
- removed the REF** at (91.0, 89.0)
- removed the REF** at (90.0, 89.0)
- removed the REF** at (89.0, 89.0)
- removed the REF** at (88.0, 89.0)
- removed the REF** at (95.0, 88.0)
- removed the REF** at (94.0, 88.0)
- removed the REF** at (93.0, 88.0)
- removed the REF** at (92.0, 88.0)
- removed the REF** at (91.0, 88.0)
- removed the REF** at (90.0, 88.0)
- removed the REF** at (89.0, 88.0)
- removed the REF** at (111.0, 94.0)
- removed the REF** at (111.0, 92.0)
- removed the REF** at (110.0, 92.0)
- removed the REF** at (106.0, 92.0)
- removed the REF** at (105.0, 92.0)
- removed the REF** at (111.0, 91.0)
- removed the REF** at (110.0, 91.0)
- removed the REF** at (106.0, 91.0)
- removed the REF** at (105.0, 91.0)
- removed the REF** at (111.0, 90.0)
- removed the REF** at (110.0, 90.0)
- removed the REF** at (106.0, 90.0)
- removed the REF** at (105.0, 90.0)
- removed the REF** at (111.0, 89.0)
- removed the REF** at (110.0, 89.0)
- removed the REF** at (106.0, 89.0)
- removed the REF** at (105.0, 89.0)
- removed the REF** at (111.0, 88.0)
- removed the REF** at (110.0, 88.0)
- removed the REF** at (106.0, 88.0)
- removed the REF** at (105.0, 88.0)
- removed the REF** at (111.0, 87.0)
- removed the REF** at (110.0, 87.0)
- removed the REF** at (109.0, 87.0)
- removed the REF** at (108.0, 87.0)
- removed the REF** at (107.0, 87.0)
- removed the REF** at (106.0, 87.0)
- removed the REF** at (105.0, 87.0)
- removed the REF** at (111.0, 86.0)
- removed the REF** at (110.0, 86.0)
- removed the REF** at (109.0, 86.0)
- removed the REF** at (108.0, 86.0)
- removed the REF** at (107.0, 86.0)
- removed the REF** at (106.0, 86.0)
- removed the REF** at (87.0, 87.0)
- removed the REF** at (86.0, 87.0)
- removed the REF** at (85.0, 87.0)
- removed the REF** at (84.0, 87.0)
- removed the REF** at (83.0, 87.0)
- removed the REF** at (87.0, 86.0)
- removed the REF** at (86.0, 86.0)
- removed the REF** at (85.0, 86.0)
- removed the REF** at (84.0, 86.0)
- removed the REF** at (83.0, 86.0)
- removed the REF** at (87.0, 85.0)
- removed the REF** at (86.0, 85.0)
- removed the REF** at (85.0, 85.0)
- removed the REF** at (84.0, 85.0)
- removed the REF** at (83.0, 85.0)
- removed the REF** at (87.0, 84.0)
- removed the REF** at (86.0, 84.0)
- removed the REF** at (87.0, 83.0)
- removed the REF** at (86.0, 83.0)
- removed the REF** at (87.0, 82.0)
- removed the REF** at (86.0, 82.0)
- removed the REF** at (87.0, 81.0)
- removed the REF** at (86.0, 81.0)
- removed the REF** at (87.0, 80.0)
- removed the REF** at (86.0, 80.0)
- removed the REF** at (87.0, 79.0)
- removed the REF** at (86.0, 79.0)
- removed the REF** at (87.0, 78.0)
- removed the REF** at (86.0, 78.0)
- removed the REF** at (87.0, 77.0)
- removed the REF** at (86.0, 77.0)
- removed the REF** at (87.0, 76.0)
- removed the REF** at (86.0, 76.0)
- removed the REF** at (87.0, 75.0)
- removed the REF** at (86.0, 75.0)
- removed the REF** at (87.0, 74.0)
- removed the REF** at (86.0, 74.0)
- removed the REF** at (87.0, 73.0)
- removed the REF** at (86.0, 73.0)
- removed the REF** at (87.0, 72.0)
- removed the REF** at (86.0, 72.0)
- removed the REF** at (87.0, 71.0)
- removed the REF** at (86.0, 71.0)
- removed the REF** at (87.0, 70.0)
- removed the REF** at (86.0, 70.0)
- removed the REF** at (87.0, 69.0)
- removed the REF** at (86.0, 69.0)
- removed the REF** at (87.0, 68.0)
- removed the REF** at (86.0, 68.0)
- removed the REF** at (87.0, 67.0)
- removed the REF** at (86.0, 67.0)
- removed the REF** at (87.0, 66.0)
- removed the REF** at (86.0, 66.0)
- removed the REF** at (87.0, 65.0)
- removed the REF** at (86.0, 65.0)
- removed the REF** at (87.0, 64.0)
- removed the REF** at (86.0, 64.0)
- removed the REF** at (87.0, 63.0)
- removed the REF** at (86.0, 63.0)
- removed the REF** at (87.0, 62.0)
- removed the REF** at (86.0, 62.0)
- removed the REF** at (87.0, 61.0)
- removed the REF** at (86.0, 61.0)
- removed the REF** at (87.0, 60.0)
- removed the REF** at (86.0, 60.0)
- removed the REF** at (87.0, 59.0)
- removed the REF** at (86.0, 59.0)
- removed the REF** at (87.0, 58.0)
- removed the REF** at (86.0, 58.0)
- removed the REF** at (87.0, 57.0)
- removed the REF** at (86.0, 57.0)
- removed the REF** at (87.0, 56.0)
- removed the REF** at (86.0, 56.0)
- removed the REF** at (87.0, 55.0)
- removed the REF** at (86.0, 55.0)
- removed the REF** at (87.0, 54.0)
- removed the REF** at (86.0, 54.0)
- removed the REF** at (85.0, 54.0)
- removed the REF** at (84.0, 54.0)
- removed the REF** at (83.0, 54.0)
- removed the REF** at (87.0, 53.0)
- removed the REF** at (86.0, 53.0)
- removed the REF** at (85.0, 53.0)
- removed the REF** at (84.0, 53.0)
- removed the REF** at (83.0, 53.0)
- removed the REF** at (105.0, 86.0)
- removed the REF** at (88.0, 88.0)
- removed the REF** at (122.0, 74.0)
- removed the REF** at (122.0, 48.0)
- removed the REF** at (121.0, 48.0)
- removed the REF** at (120.0, 48.0)
- removed the REF** at (119.0, 48.0)
- removed the REF** at (118.0, 48.0)
- removed the REF** at (117.0, 48.0)
- removed the REF** at (116.0, 48.0)
- removed the REF** at (115.0, 48.0)
- removed the REF** at (114.0, 48.0)
- removed the REF** at (113.0, 48.0)
- removed the REF** at (112.0, 48.0)
- removed the REF** at (111.0, 48.0)
- removed the REF** at (110.0, 48.0)
- removed the REF** at (109.0, 48.0)
- removed the REF** at (108.0, 48.0)
- removed the REF** at (107.0, 48.0)
- removed the REF** at (106.0, 48.0)
- removed the REF** at (105.0, 48.0)
- removed the REF** at (104.0, 48.0)
- removed the REF** at (103.0, 48.0)
- removed the REF** at (102.0, 48.0)
- removed the REF** at (101.0, 48.0)
- removed the REF** at (100.0, 48.0)
- removed the REF** at (99.0, 48.0)
- removed the REF** at (98.0, 48.0)
- removed the REF** at (97.0, 48.0)
- removed the REF** at (96.0, 48.0)
- removed the REF** at (95.0, 48.0)
- removed the REF** at (94.0, 48.0)
- added J2: Conn_01x01, MountingHole:MountingHole_3.2mm_M3_ISO14580_Pad, F.Cu at (84.0, 49.0)
- added REF**: via, via:via, F.Cu at (122.0, 94.0)
- added REF**: via, via:via, F.Cu at (113.0, 94.0)
- added REF**: via, via:via, F.Cu at (112.0, 94.0)
- added REF** (x2): via, via:via, F.Cu at (111.0, 94.0)
- added REF**: via, via:via, F.Cu at (122.0, 93.0)
- added REF**: via, via:via, F.Cu at (121.0, 93.0)
- added REF**: via, via:via, F.Cu at (120.0, 93.0)
- added REF**: via, via:via, F.Cu at (119.0, 93.0)
- added REF**: via, via:via, F.Cu at (118.0, 93.0)
- added REF**: via, via:via, F.Cu at (117.0, 93.0)
- added REF**: via, via:via, F.Cu at (116.0, 93.0)
- added REF**: via, via:via, F.Cu at (121.0, 94.0)
- added REF**: via, via:via, F.Cu at (115.0, 93.0)
- added REF**: via, via:via, F.Cu at (114.0, 93.0)
- added REF**: via, via:via, F.Cu at (113.0, 93.0)
- added REF**: via, via:via, F.Cu at (112.0, 93.0)
- added REF**: via, via:via, F.Cu at (120.0, 94.0)
- added REF**: via, via:via, F.Cu at (119.0, 94.0)
- added REF**: via, via:via, F.Cu at (118.0, 94.0)
- added REF**: via, via:via, F.Cu at (117.0, 94.0)
- added REF**: via, via:via, F.Cu at (116.0, 94.0)
- added REF**: via, via:via, F.Cu at (115.0, 94.0)
- added REF**: via, via:via, F.Cu at (114.0, 94.0)
Routing:
- net Net-(J3-Pad1): track 24.6 -> 21.6 mm
- net GND: track 106.2 -> 104.2 mm

Commit message: new iBom
Other:
- net class Default removed
